Commit message: Camera positions in the URDF, keyboard-drivable simulation
- Camera positions now live in wizja_description/urdf/wizja_rover.urdf.xacro
  (CAMERA POSITIONS block, tripod-screw poses like rover30); cameras.yaml only
  lists which cameras exist; launch/tools check every yaml camera is placed
- sim_drive.launch.py: drive the simulated rover with teleop_twist_keyboard
  (4-wheel steering kinematics, animated steer/wheel joints, odom TF, /odom,
  ground-truth scene markers, follow-camera RViz config)
- Faster simulator renderer: analytic ground + Lipschitz-safe hill march,
  cached rover occlusion, culling, decimated front-camera rendering
- Tests for the steering/pose kinematics and URDF camera placement

Co-Authored-By: Claude Opus 5.5 <noreply@anthropic.com>

File: src/wizja_description/urdf/wizja_rover.urdf.xacro (robot description, xacro)
@@ -1,24 +1,24 @@
 <?xml version="1.0"?>
 <!--
-  Rover 3.0 (rover30) visual model with the depth-camera cluster of lr_wizja_kamery.
+  Rover 3.0 (rover30) visual model with the depth cameras of lr_wizja_kamery.
+  >>> CAMERA POSITIONS ARE EDITED IN THIS FILE: see the "CAMERA POSITIONS" block below. <<<
+  After editing, rebuild the wizja_description package (exact commands in README, "Changing camera
+  positions"), then check with view_model.launch.py and coverage_map.py.
+  wizja_bringup/config/cameras.yaml only says WHICH cameras exist (serials, driver/external, topics);
+  every camera listed there must be placed here under its frame prefix (camera_<name>, or its
+  frame_prefix), otherwise the launch files stop with an error.
   Rover geometry, joint origins/limits and meshes are taken from Aut-Main rover30_description
-  (rover30_ASSEMBLY_NEW.urdf.xacro, simplified meshes). The lidar and the old front vision D455 are
-  left out: they are replaced by the camera cluster below.
+  (rover30_ASSEMBLY_NEW.urdf.xacro, simplified meshes). The lidar is left out: the cameras replace it.
   Args:
-    cameras_config         wizja_bringup cameras.yaml (camera names + base_link -> camera_<name>_link poses)
     include_rover          true:  full model, root base_footprint (standalone / laptop / simulator)
-                           false: only base_link + camera mount + cameras, for running next to the main
-                                  rover stack whose robot_state_publisher already publishes the rover
-    nominal_camera_frames  true: also add <prefix>_depth_frame / _depth_optical_frame. Only for
+                           false: only base_link + camera post + side cameras, for running next to the
+                                  main rover stack whose robot_state_publisher already publishes the
+                                  rover and the front camera (camera_link ...)
+    nominal_camera_frames  true: also add <name>_depth_frame / _depth_optical_frame. Only for
                            the simulator - on hardware the realsense driver publishes them (publish_tf).
-  Cameras with `source: external` in cameras.yaml (the rover's front D455, owned by the main stack)
-  are only added when include_rover=true; with include_rover=false the main stack's URDF already
-  publishes their frames (camera_link, ...).
 -->
 <robot name="rover30_wizja" xmlns:xacro="http://ros.org/wiki/xacro">
-  <xacro:arg name="cameras_config" default="$(find wizja_bringup)/config/cameras.yaml"/>
   <xacro:arg name="include_rover" default="true"/>
   <xacro:arg name="nominal_camera_frames" default="false"/>
-  <xacro:property name="rig" value="${xacro.load_yaml('$(arg cameras_config)')}"/>
   <xacro:property name="include_rover" value="${'$(arg include_rover)'.lower() in ('true', '1')}"/>
   <xacro:property name="nominal_frames" value="${'$(arg nominal_camera_frames)'.lower() in ('true', '1')}"/>
@@ -28,9 +28,68 @@
   <!-- Top of the deck in base_link (measured from base_link.stl) -->
   <xacro:property name="deck_top_z" value="0.18"/>
-  <!-- Camera post for the side cameras: where the lidar used to be (rover30 laser_joint xyz 0.33 0 0.185) -->
+  <!-- Camera post for the side cameras: where the lidar used to be (rover30 laser_joint xyz 0.33 0 0.185).
+       Visual only (+ simulator occlusion box in wizja_bringup/rover_geometry.py). -->
   <xacro:property name="post_x" value="0.33"/>
   <xacro:property name="post_y" value="0.0"/>
   <xacro:property name="post_height" value="0.20"/>
   <xacro:property name="post_radius" value="0.02"/>
+  <!-- One D455, placed by its tripod-screw frame (bottom centre of the camera = what you measure).
+       <name>_link = realsense body frame (X out of the lens, origin at the left IR imager = depth
+       origin), the frame realsense2_camera hangs its optical frames on. Offsets and visual from
+       rover30 include/rs_d455.urdf.xacro. Do not edit - edit the CAMERA POSITIONS block below. -->
+  <xacro:macro name="d455" params="name parent xyz rpy">
+    <joint name="${name}_joint" type="fixed">
+      <parent link="${parent}"/>
+      <child link="${name}_bottom_screw_frame"/>
+      <origin xyz="${xyz}" rpy="${rpy}"/>
+    </joint>
+    <link name="${name}_bottom_screw_frame"/>
+    <joint name="${name}_link_joint" type="fixed">
+      <parent link="${name}_bottom_screw_frame"/>
+      <child link="${name}_link"/>
+      <origin xyz="0.01115 0.0475 0.0145" rpy="0 0 0"/>
+    </joint>
+    <link name="${name}_link">
+      <visual>
+        <origin xyz="${4.55e-3 + 0.1e-3} -0.0475 0" rpy="${pi/2} 0 ${pi/2}"/>
+        <geometry><mesh filename="${mesh_dir}/rs_d455.stl" scale="0.001 0.001 0.001"/></geometry>
+        <material name="aluminum"/>
+      </visual>
+    </link>
+    <xacro:if value="${nominal_frames}">
+      <joint name="${name}_depth_joint" type="fixed">
+        <parent link="${name}_link"/>
+        <child link="${name}_depth_frame"/>
+        <origin xyz="0 0 0" rpy="0 0 0"/>
+      </joint>
+      <link name="${name}_depth_frame"/>
+      <joint name="${name}_depth_optical_joint" type="fixed">
+        <parent link="${name}_depth_frame"/>
+        <child link="${name}_depth_optical_frame"/>
+        <origin xyz="0 0 0" rpy="${-pi/2} 0 ${-pi/2}"/>
+      </joint>
+      <link name="${name}_depth_optical_frame"/>
+    </xacro:if>
+  </xacro:macro>
+  <!-- ================================== CAMERA POSITIONS ==================================
+       xyz = position of the camera's TRIPOD SCREW (bottom centre of the D455) in base_link:
+             x forward, y left, z up, metres. base_link = rover centre, 0.38 m above the ground,
+             deck top at z = 0.18.
+       rpy = roll pitch yaw in radians (URDF convention): pitch > 0 tilts the camera DOWN,
+             yaw > 0 turns it to the LEFT (+1.5708 = facing left, -1.5708 = facing right).
+       The camera's depth origin (<name>_link) is 1.1 cm in front of, 4.75 cm left of and
+       1.45 cm above the screw (in the camera's own frame).
+       ======================================================================================= -->
+  <!-- Left / right: our drivers, on the post where the lidar used to be. Yaw +/-80 deg (not 90) so
+       the front diagonals overlap with the front camera; 20 deg down. DESIGN VALUES - measure after
+       mounting. -->
+  <xacro:d455 name="camera_left"  parent="base_link" xyz="0.28910 0.08254 0.38520" rpy="0 0.35 1.3963"/>
+  <xacro:d455 name="camera_right" parent="base_link" xyz="0.28854 -0.08304 0.38520" rpy="0 0.35 -1.3963"/>
+  <!-- Front ("Center"): the rover's existing D455, owned by the main stack, which publishes its TF
+       from Aut-Main rover30_description (camera_joint). Only added in the full model; if it is moved,
+       change it HERE AND in rover30_description so both stay equal. -->
+  <xacro:if value="${include_rover}">
+    <xacro:d455 name="camera" parent="base_link" xyz="0.42 0.0 0.18" rpy="0 0 0"/>
+  </xacro:if>
   <material name="purple"><color rgba="${114/255} 0 1 1"/></material>
   <material name="steer_blue"><color rgba="${202/255} ${209/255} ${238/255} 1"/></material>
@@ -109,47 +168,3 @@
     <origin xyz="${post_x} ${post_y} ${deck_top_z}" rpy="0 0 0"/>
   </joint>
-  <!-- One D455. camera_<name>_link = realsense body frame (X out of the lens, origin at the left IR
-       imager = depth origin), exactly the frame realsense2_camera hangs its optical frames on. Visual
-       offsets from rover30 include/rs_d455.urdf.xacro. -->
-  <xacro:macro name="d455" params="name parent pose">
-    <joint name="${name}_mount_joint" type="fixed">
-      <parent link="${parent}"/>
-      <child link="${name}_link"/>
-      <origin xyz="${pose['x']} ${pose['y']} ${pose['z']}" rpy="${pose['roll']} ${pose['pitch']} ${pose['yaw']}"/>
-    </joint>
-    <link name="${name}_link">
-      <visual>
-        <origin xyz="${4.55e-3 + 0.1e-3} -0.0475 0" rpy="${pi/2} 0 ${pi/2}"/>
-        <geometry><mesh filename="${mesh_dir}/rs_d455.stl" scale="0.001 0.001 0.001"/></geometry>
-        <material name="aluminum"/>
-      </visual>
-    </link>
-    <xacro:if value="${nominal_frames}">
-      <joint name="${name}_depth_joint" type="fixed">
-        <parent link="${name}_link"/>
-        <child link="${name}_depth_frame"/>
-        <origin xyz="0 0 0" rpy="0 0 0"/>
-      </joint>
-      <link name="${name}_depth_frame"/>
-      <joint name="${name}_depth_optical_joint" type="fixed">
-        <parent link="${name}_depth_frame"/>
-        <child link="${name}_depth_optical_frame"/>
-        <origin xyz="0 0 0" rpy="${-pi/2} 0 ${-pi/2}"/>
-      </joint>
-      <link name="${name}_depth_optical_frame"/>
-    </xacro:if>
-  </xacro:macro>
-  <!-- Iterate over the cameras of cameras.yaml (xacro has no loops -> recursion over the name list) -->
-  <xacro:macro name="cameras" params="names">
-    <xacro:if value="${len(names) > 0}">
-      <xacro:property name="cam" value="${rig['cameras'][names[0]]}"/>
-      <xacro:if value="${include_rover or cam.get('source', 'driver') != 'external'}">
-        <xacro:d455 name="${cam.get('frame_prefix', '') or 'camera_' + names[0]}"
-                    parent="${rig.get('parent_frame', 'base_link')}"
-                    pose="${cam['pose']}"/>
-      </xacro:if>
-      <xacro:cameras names="${names[1:]}"/>
-    </xacro:if>
-  </xacro:macro>
-  <xacro:cameras names="${list(rig['cameras'].keys())}"/>
 </robot>
